File: hw/hw.kicad_sch (KiCad schematic)
At the start: 44 parts, among them CN1 PJ-320D, U1 ICE40LP1K-QN84, U2 MAX98357AETE+T, U5 AP2112K-3.3, U6 AP2112K-1.8, U6 AT25SF081-SSHD-X, U7 MIC5219-2.8YM5, U7 YF4016M00033T8188092, U8 PM004MNIATR

Commit message: switch to a fpga with more gpio + doc
Parts:
- removed C1: C, Capacitor_SMD:C_0402_1005Metric, symbol Device:C
- removed U1: ICE40LP1K-QN84, footprint:LATTICE_ICE40LP1K-QN84, symbol ICE40LP1K-QN84:ICE40LP1K-QN84
- removed USB2: 12401832E402A, easyeda2kicad:USB-C-TH_12401832E402A, symbol easyeda2kicad:12401832E402A
- added C10, C11, C16, C9: 100nF, Capacitor_SMD:C_0201_0603Metric, symbol TinyFPGA-BX-rescue:C_Small
- added C12, C13, C14, C15: 10nF, Capacitor_SMD:C_0201_0603Metric, symbol TinyFPGA-BX-rescue:C_Small
- added C17, C6: 10uF, Capacitor_SMD:C_0402_1005Metric, symbol TinyFPGA-BX-rescue:C
- added C2, C3: 1uF, Capacitor_SMD:C_0402_1005Metric, symbol TinyFPGA-BX-rescue:C
- added C2 (x2): 22uF, Capacitor_SMD:C_0402_1005Metric, symbol Device:C
- added C5, C7, C8: 100nF, Capacitor_SMD:C_0201_0603Metric, symbol TinyFPGA-BX-rescue:C
- added L1: Bead, Inductor_SMD:L_0603_1608Metric, symbol TinyFPGA-BX-rescue:Ferrite_Bead_Small
- added R1: 1.5k, Resistor_SMD:R_0201_0603Metric, symbol TinyFPGA-BX-rescue:R
- added R10, R5, R7: 10k, Resistor_SMD:R_0201_0603Metric, symbol TinyFPGA-BX-rescue:R
- added R14: 0R, Capacitor_SMD:C_0402_1005Metric, symbol Device:R
- added R16: 5.1K, Resistor_SMD:R_0201_0603Metric, symbol Device:R
- added R2, R3: 68, Resistor_SMD:R_0201_0603Metric, symbol TinyFPGA-BX-rescue:R
- added R4: 100, Resistor_SMD:R_0201_0603Metric, symbol TinyFPGA-BX-rescue:R
- added R6: R, Resistor_SMD:R_0201_0603Metric, symbol TinyFPGA-BX-rescue:R
- added SW1: SW_Push, tinyfpga:PTS_810_SMT_Switch, symbol TinyFPGA-BX-rescue:SW_Push
- added TP1, TP2, TP3: TEST, TestPoint:TestPoint_Pad_D1.0mm, symbol TinyFPGA-BX-rescue:TEST
- added U1: ICE40LP8K-CM121, footprint:BGA121N40P11X11_500X500X100N, symbol ICE40LP8K-CM121:ICE40LP8K-CM121
- added U4: MIC5365-1.2YC5-TR, tinyfpga:SC-70-C5, symbol TinyFPGA-BX-rescue:MIC5365-1.2YC5-TR
- C52, C55, C57: footprint Capacitor_SMD:C_0402_1005Metric -> Capacitor_SMD:C_0201_0603Metric
- D4: footprint (none) -> Diode_SMD:D_0402_1005Metric
- R1: value R -> 5.1K; footprint Resistor_SMD:R_0402_1005Metric -> Resistor_SMD:R_0201_0603Metric
- R17, R18, R19, R20: footprint Capacitor_SMD:C_0402_1005Metric -> Resistor_SMD:R_0201_0603Metric
Connections:
- net +1V2: now also C11.1, C12.1, C13.1, C3.1, R4.2, TP3.1, U1.D4 (VCC), U1.D8 (VCC__1), U1.G1 (IOL_14A_GBIN6), U1.H4 (VCC__2), U1.H8 (VCC__3), U4.5 (VOUT)
- net +3.3V: now also U6.8 (VCC), C10.1, C14.1, C15.1, C16.1, C9.1, R10.1, R7.1
- net DVP0_HREF: now also U1.H1 (IOL_18A)
- net DVP0_MCLK: now also U1.A3 (IOT_223)
- net DVP0_PCLK: now also U1.F4 (IOL_13A)
- net DVP0_SCL: now also U1.D10 (IOR_154)
- net DVP0_SDA: now also U1.D11 (IOR_152)
- net DVP0_VSYNC: now also U1.H3 (IOL_17B)
- net DVP0_Y2: now also U1.J1 (IOL_23A)
- net DVP0_Y3: now also U1.K2 (IOL_25A)
- net DVP0_Y4: now also U1.J2 (IOL_25B)
- net DVP0_Y5: now also U1.K1 (IOL_23B)
- net DVP0_Y6: now also U1.H2 (IOL_18B)
- net DVP0_Y7: now also U1.F2 (IOL_12B)
- net DVP0_Y8: now also U1.A1 (IOT_225)
- net DVP0_Y9: now also U1.L4 (IOB_72)
- net DVP1_HREF: now also U1.D7 (IOT_181)
- net DVP1_MCLK: now also U1.D5 (IOT_212)
- net DVP1_PCLK: now also U1.L1 (IOB_56)
- net DVP1_SCL: now also U1.E11 (IOR_148)
- net DVP1_SDA: now also U1.D9 (IOR_147)
- net DVP1_VSYNC: now also U1.A5 (IOT_207)
- net DVP1_Y2: now also U1.K3 (IOB_63)
- net DVP1_Y3: now also U1.L3 (IOB_71)
- net DVP1_Y4: now also U1.G3 (IOL_17A)
- net DVP1_Y5: now also U1.J4 (IOB_64)
- net DVP1_Y6: now also U1.L2 (IOB_61)
- net DVP1_Y7: now also U1.J3 (IOB_57)
- net DVP1_Y8: now also U1.B4 (IOT_219)
- net DVP1_Y9: now also U1.A8 (IOT_190)
- net DVP2_MCLK: now also U1.B11 (IOR_161)
- net DVP2_PCLK: now also U1.A6 (IOT_206)
- net DVP2_SCL: now also U1.E8 (IOR_146)
- net DVP2_SDA: now also U1.E9 (IOR_144)
- net DVP2_VSYNC: now also U1.C11 (IOR_160)
- net DVP2_Y2: now also U1.A2 (IOT_222)
- net DVP2_Y3: now also U1.B3 (IOT_221)
- net DVP2_Y4: now also U1.A7 (IOT_192)
- net DVP2_Y5: now also U1.C7 (IOT_191)
- net DVP2_Y6: now also U1.H11 (IOR_119)
- net DVP2_Y7: now also U1.F1 (IOL_12A)
- net DVP2_Y8: now also U1.G8 (IOR_118)
- net DVP2_Y9: now also U1.J10 (IOR_117)
- net GND: now also R1.2, USB1.0, C10.2, C11.2, C12.2, C13.2, C14.2, C15.2, C16.2, C17.1, C2.2, C2.2, C2.2, C3.2, C5.2, C8.2, C9.2, L1.1, R16.2, SW1.1, U1.B1 (IOL_2A), U1.B9 (IOT_174), U1.E5 (GND), U1.E6 (GND__1), U1.E7 (GND__2), U1.F5 (GND__3), U1.F6 (GND__4), U1.F7 (GND__5), U1.G2 (IOL_14B), U1.G5 (GND__6), U1.G6 (GND__7), U1.G7 (GND__8), U1.H5 (GND__9), U4.2 (GND)
- net VBUS: now also U6.1 (VIN), U6.3 (EN), U7.1 (IN), U7.3 (EN), USB1.A4 (VBUS), USB1.A9 (VBUS), USB1.B4 (VBUS), USB1.B9 (VBUS), C17.2, C2.1, C2.1, L1.2
- net SS: now reaches U6.1 (~{CS})
- net SS: now also R5.2, U1.K10 (IOB_108_SS), U1.K11 (IOR_115)
- net SDI: now reaches U6.2 (SO/IO1)
- net SDI: now also U1.J9 (IOB_106_SDI)
- net 82: now reaches U6.3 (~{WP}/IO2)
- net 82: now also R7.2, TP1.1, U1.K6 (IOB_82_GBIN4)
- net SDO: now reaches U6.5 (SI/IO0)
- net SDO: now also U1.H9 (IOB_104_CBSEL1), U1.K9 (IOB_105_SDO)
- net SCK: now reaches U6.6 (SCK)
- net SCK: now also U1.J11 (IOR_114), U1.L10 (IOB_107_SCK)
- net 109: now reaches U6.7 (~{HOLD}/IO3)
- net 109: now also R10.2, U1.H10 (IOR_116)
- net at U7.1 (Tri-state): now also R14.2
- net CLK: now reaches U7.3 (Output)
- net CLK: now also U1.B2 (IOL_2B)
- net +3V3: now reaches U7.4 (Vdd)
- net +3V3: now also C2.1, C5.1, C8.1, R14.1, R5.1, R6.1, U1.B8 (IOT_177), U1.C10 (VPP_2V5), U1.D6 (VCCIO_0), U1.E4 (VCCIO_3), U1.F8 (VCCIO_1), U1.G10 (IOR_120), U1.G4 (VCCIO_3__1), U1.H6 (VCCIO_2), U1.L11 (VCC_SPI), U4.1 (VIN), U4.3 (EN)
- net at USB1.A5 (CC1): now also R16.1
- net USB_D_P: now reaches USB1.A6 (D+)
- net USB_D_P: now also USB1.B6 (D+), R1.1, R2.2
- net USB_D_N: now reaches USB1.A7 (D-)
- net USB_D_N: now also USB1.B7 (D-), R3.2
- net at USB1.B5 (CC2): now also R1.1
- new net: C6.1, C7.1, R4.1, U1.C6 (VCCPLL1), U1.J6 (VCCPLL0)
- new net: C6.2, C7.2, U1.C5 (GNDPLL1), U1.L6 (GNDPLL0)
- new net CDONE: U1.K8 (CDONE)
- new net CRESET_B: R6.2, SW1.2, TP2.1, U1.L9 (~{CRESET})
- new net USB_N: R3.1, U1.B5 (IOT_208)
- new net USB_P: R2.1, U1.A4 (IOT_211)
- new net USB_PU: R1.2, U1.A9 (IOT_178)
- new net VPP_FAST: U1.B10 (VPP_FAST)
- no-connect marks 3 -> 13
Other:
- note added: "16MHz Clock"
- note added: "FPGA PLL decoupling capacitors"
- note added: "FPGA connections"
- note added: "FPGA core and IO power connections and decoupling capacitors"
- note added: "FPGA reset button and testpoint"
- note added: "SPI flash memory for FPGA configuration"
- note added: "Voltage Regulation"
- moved on the sheet: C1, C2, R1, U2, U5, U6, U7, U8, USB1
